Commit message: ur5 fix

File: robot_urdf/generated_urdf/ur5.urdf (robot description, URDF)
Before this commit: robot ur_robot, 35 links, 34 joints
Links:
- added link gripper_base; collision mesh filename=package://gripper_description/meshes/gripper_base_up.stl scale=0.001 0.001 0.001; visual mesh filename=package://gripper_description/meshes/gripper_base_up.stl scale=0.001 0.001 0.001
- added link gripper_base_down, mass 1.0; collision mesh filename=package://gripper_description/meshes/gripper_base_down.stl scale=0.001 0.001 0.001; visual mesh filename=package://gripper_description/meshes/gripper_base_down.stl scale=0.001 0.001 0.001
- added link hand_1_link, mass 0.05; collision mesh filename=package://gripper_description/meshes/finger.stl scale=0.001 0.001 0.001; visual mesh filename=package://gripper_description/meshes/finger.stl scale=0.001 0.001 0.001
- added link hand_2_link, mass 0.05; collision mesh filename=package://gripper_description/meshes/finger.stl scale=0.001 0.001 0.001; visual mesh filename=package://gripper_description/meshes/finger.stl scale=0.001 0.001 0.001
- added link hand_3_link, mass 0.05; collision mesh filename=package://gripper_description/meshes/finger.stl scale=0.001 0.001 0.001; visual mesh filename=package://gripper_description/meshes/finger.stl scale=0.001 0.001 0.001
- added link tool0_without_gripper
Joints:
- removed joint ee_camera/tool0camera_joint
- added joint ee_camera/wrist_3_linkcamera_joint: type fixed, parent wrist_3_link, child ee_camera/camera_bottom_screw_frame, origin xyz=0.05 0.0 -0.02 rpy=0 -1.57 0.0
- added joint fixed_ee_gripper: type fixed, parent gripper_base, child tool0, origin xyz=0 0 0.12 rpy=0 0 0
- added joint flange: type fixed, parent gripper_base, child gripper_base_down, origin xyz=0 0 0.06 rpy=0 0 0
- added joint gripper_robot_joint: type fixed, parent tool0_without_gripper, child gripper_base, origin xyz=0 0 0 rpy=0 0 3.14
- added joint hand_1_joint: type fixed, parent gripper_base_down, child hand_1_link, origin xyz=0.0  -0.03 0.05 rpy=-1.5707963267948966 0 0
- added joint hand_2_joint: type fixed, parent gripper_base_down, child hand_2_link, origin xyz=0.02598 0.015 0.05 rpy=-1.5707963267948966 0 2.0943951023931953
- added joint hand_3_joint: type fixed, parent gripper_base_down, child hand_3_link, origin xyz=-0.02598 0.015 0.05 rpy=-1.5707963267948966 0 -2.0943951023931953
- joint flange-tool0: child tool0 -> tool0_without_gripper
- joint z_base_camera/base_linkcamera_joint: origin xyz=0.0 -0.3 -0.5 rpy=0.0  0.5 1.57 -> xyz=0.0 1.0 -0.25 rpy=3.14  -4.0 1.57
