Commit message: moved the camera

File: robot_descriptions/ur_description/urdf/ur5.urdf.xacro (robot description, xacro)
@@ -57,8 +57,8 @@
 		<origin xyz="0.05 0.0 -0.02" rpy="0 -1.57 0.0"/>
 	</xacro:d435_camera>
-	  <xacro:property name="camera_fov" value="3.0"/>
+	  <xacro:property name="camera_fov" value="1.5"/>
 	  <xacro:property name="camera_width" value="640"/>
 	  <xacro:property name="camera_height" value="480"/>
-	  <xacro:property name="camera_near" value="0.01"/>
+	  <xacro:property name="camera_near" value="0.60"/>
 	  <xacro:property name="camera_far" value="100"/>
 	<xacro:d435_camera
@@ -66,5 +66,6 @@
 		name="z_base_camera"
 		camera_plugin="true">
-		<origin xyz="0.0 -0.3 -0.5" rpy="0.0  0.5 1.57"/>
+		<!--<origin xyz="0.0 -0.3 -0.5" rpy="0.0  0.5 1.57"/> -->
+		<origin xyz="0.0 1.0 -0.25" rpy="3.14  -4.0 1.57"/>
 	</xacro:d435_camera>
 </xacro:if>

Commit message: fixed bugs

File: robot_descriptions/ur_description/urdf/ur5.urdf.xacro (robot description, xacro)
@@ -57,8 +57,8 @@
 		<origin xyz="0.05 0.0 -0.02" rpy="0 -1.57 0.0"/>
 	</xacro:d435_camera>
-	  <xacro:property name="camera_fov" value="1.5"/>
+	  <xacro:property name="camera_fov" value="3.0"/>
 	  <xacro:property name="camera_width" value="640"/>
 	  <xacro:property name="camera_height" value="480"/>
-	  <xacro:property name="camera_near" value="0.60"/>
+	  <xacro:property name="camera_near" value="0.01"/>
 	  <xacro:property name="camera_far" value="100"/>
 	<xacro:d435_camera
@@ -66,6 +66,5 @@
 		name="z_base_camera"
 		camera_plugin="true">
-		<!--<origin xyz="0.0 -0.3 -0.5" rpy="0.0  0.5 1.57"/> -->
-		<origin xyz="0.0 1.0 -0.25" rpy="3.14  -4.0 1.57"/>
+		<origin xyz="0.0 -0.3 -0.5" rpy="0.0  0.5 1.57"/>
 	</xacro:d435_camera>
 </xacro:if>

File: robot_urdf/generated_urdf/ur5.urdf (robot description, URDF)
Before this commit: robot ur_robot, 41 links, 40 joints
Joints:
- joint z_base_camera/base_linkcamera_joint: origin xyz=0.0 1.0 -0.25 rpy=3.14  -4.0 1.57 -> xyz=0.0 -0.3 -0.5 rpy=0.0  0.5 1.57

Commit message: Changed cam position

File: robot_descriptions/ur_description/urdf/ur5.urdf.xacro (robot description, xacro)
@@ -57,8 +57,8 @@
 		<origin xyz="0.05 0.0 -0.02" rpy="0 -1.57 0.0"/>
 	</xacro:d435_camera>
-	  <xacro:property name="camera_fov" value="3.0"/>
+	  <xacro:property name="camera_fov" value="1.5"/>
 	  <xacro:property name="camera_width" value="640"/>
 	  <xacro:property name="camera_height" value="480"/>
-	  <xacro:property name="camera_near" value="0.01"/>
+	  <xacro:property name="camera_near" value="0.6"/>
 	  <xacro:property name="camera_far" value="100"/>
 	<xacro:d435_camera
@@ -66,5 +66,5 @@
 		name="z_base_camera"
 		camera_plugin="true">
-		<origin xyz="0.0 -0.3 -0.5" rpy="0.0  0.5 1.57"/>
+		<origin xyz="0.0 1.0 -0.25" rpy="3.14 -4.0 1.57"/>
 	</xacro:d435_camera>
 </xacro:if>

File: robot_urdf/generated_urdf/ur5.urdf (robot description, URDF)
Before this commit: robot ur_robot, 41 links, 40 joints
Joints:
- joint z_base_camera/base_linkcamera_joint: origin xyz=0.0 -0.3 -0.5 rpy=0.0  0.5 1.57 -> xyz=0.0 1.0 -0.25 rpy=3.14 -4.0 1.57
